Commit message: make the urdf and xml similar. rotate the reference frame for each link

File: open-chain.urdf (robot description, URDF)
Before this commit: robot open-chain, 6 links, 5 joints
Links:
- removed link ee_link
- added link end_effector; visual sphere radius=0.05
Joints:
- joint ee_joint: child ee_link -> end_effector

Commit message: fix center of mass position in urdf file

File: open-chain.urdf (robot description, URDF)
Before this commit: robot open-chain, 6 links, 5 joints
Links:
- link base_link: mass 0.5 -> None; geometry 
